Commit message: refactor(bringup): move joint_limits.yaml into omx_bringup share, document URDF fork
- copy joint_limits.yaml from upstream into omx_bringup/config/omx_f/ so
  every MoveIt config is colocated; omx_moveit.launch.py now resolves
  it via get_package_share_directory instead of a Path('config') hack
- align omx_f_with_camera.urdf.xacro port_name default with launch
  (ttyACM0, was ttyACM1 — launch arg always overrode it but the mismatch
  was confusing when reading xacro alone)
- rewrite the in-file comment block to explain why we copied upstream
  omx_f.urdf.xacro's world / end_effector_* skeleton (we cannot include
  upstream's top-level xacro because it would also pull in
  omx_f.ros2_control.xacro and clash with our grasp ros2_control)

Co-Authored-By: Claude Opus 4.7 <noreply@anthropic.com>

File: src/omx_bringup/config/omx_f/omx_f_with_camera.urdf.xacro (robot description, xacro)
@@ -7,47 +7,49 @@
   <xacro:arg name="config_type" default="omx_f" />
   <xacro:arg name="ros2_control_type" default="omx_f" />
-  <xacro:arg name="port_name" default="/dev/ttyACM1" />
+  <xacro:arg name="port_name" default="/dev/ttyACM0" />
+  <!--
+    upstream open_manipulator_description/urdf/omx_f/omx_f.urdf.xacro 의
+    world / end_effector_* 를 그대로 가져온 것.
+    upstream 최상위를 통째로 include 하면 omx_f.ros2_control.xacro 도 같이
+    들어와 우리 grasp ros2_control 과 충돌하므로, 뼈대만 복사해서
+    ros2_control include 만 omx_f_grasp.ros2_control.xacro 로 교체했다.
+  -->
   <xacro:include filename="$(find open_manipulator_description)/gazebo/omx_f.gazebo.xacro" />
   <xacro:include filename="$(find open_manipulator_description)/urdf/omx_f/omx_f_arm.urdf.xacro" />
-  <!--
-    grasp detection (effort state + Present Current) 노출용 자체 ros2_control xacro.
-    upstream open_manipulator_description/ros2_control/omx_f.ros2_control.xacro 를
-    omx_bringup/config/omx_f/omx_f_grasp.ros2_control.xacro 로 대체한다.
-  -->
   <xacro:include filename="$(find omx_bringup)/config/omx_f/omx_f_grasp.ros2_control.xacro" />
-  <link name="world"/>
+  <link name="world" />
   <joint name="$(arg prefix)world_fixed" type="fixed">
-    <parent link="world"/>
-    <child link="$(arg prefix)link0"/>
-    <origin xyz="0.0 0.0 0.0" rpy="0 0 0"/>
+    <parent link="world" />
+    <child link="$(arg prefix)link0" />
+    <origin xyz="0.0 0.0 0.0" rpy="0 0 0" />
   </joint>
   <joint name="$(arg prefix)end_effector_joint" type="fixed">
-    <parent link="$(arg prefix)link5"/>
-    <child link="$(arg prefix)end_effector_link"/>
-    <origin xyz="0.09193 -0.0016 0" rpy="0 0 0"/>
+    <parent link="$(arg prefix)link5" />
+    <child link="$(arg prefix)end_effector_link" />
+    <origin xyz="0.09193 -0.0016 0" rpy="0 0 0" />
   </joint>
   <link name="$(arg prefix)end_effector_link">
     <visual>
-      <origin xyz="0 0 0" rpy="0 0 0"/>
+      <origin xyz="0 0 0" rpy="0 0 0" />
       <geometry>
         <box size="0.01 0.01 0.01" />
       </geometry>
       <material name="red">
-        <color rgba="1.0 0.0 0.0 1"/>
+        <color rgba="1.0 0.0 0.0 1" />
       </material>
     </visual>
   </link>
   <!-- Camera frames previously published via static_transform_publisher. -->
-  <link name="$(arg prefix)camera_mount"/>
+  <link name="$(arg prefix)camera_mount" />
   <joint name="$(arg prefix)camera_mount_joint" type="fixed">
-    <parent link="$(arg prefix)link5"/>
-    <child link="$(arg prefix)camera_mount"/>
-    <origin xyz="0.025 0.0 0.054" rpy="0.0 0.65 0.0"/>
+    <parent link="$(arg prefix)link5" />
+    <child link="$(arg prefix)camera_mount" />
+    <origin xyz="0.025 0.0 0.054" rpy="0.0 0.65 0.0" />
   </joint>
-  <link name="$(arg prefix)default_cam"/>
+  <link name="$(arg prefix)default_cam" />
   <joint name="$(arg prefix)default_cam_joint" type="fixed">
-    <parent link="$(arg prefix)camera_mount"/>
-    <child link="$(arg prefix)default_cam"/>
-    <origin xyz="0.0312 0.0 0.0" rpy="-1.5708 0.0 -1.5708"/>
+    <parent link="$(arg prefix)camera_mount" />
+    <child link="$(arg prefix)default_cam" />
+    <origin xyz="0.0312 0.0 0.0" rpy="-1.5708 0.0 -1.5708" />
   </joint>
   <xacro:omx_f prefix="$(arg prefix)" />
@@ -57,8 +59,9 @@
     use_mock_hardware="$(arg use_mock_hardware)"
     mock_sensor_commands="$(arg mock_sensor_commands)"
-    port_name="$(arg port_name)"/>
+    port_name="$(arg port_name)" />
   <gazebo>
     <plugin filename="gz_ros2_control-system" name="gz_ros2_control::GazeboSimROS2ControlPlugin">
-      <parameters>$(find open_manipulator_bringup)/config/$(arg config_type)/hardware_controller_manager.yaml</parameters>
+      <parameters>$(find open_manipulator_bringup)/config/$(arg
+        config_type)/hardware_controller_manager.yaml</parameters>
     </plugin>
   </gazebo>
